File: hardware/uven-mainboard/uven-mainboard.sch (KiCad schematic (older format))
At the start: 29 parts, among them J1 TEMP_LED0, J2 TEMP_LED1, J3 TEMP_LED2, J4 TEMP_LED3, J5 TEMP_LED4, J6 LED_CONTROL, Q1 2N7002, U1 TLI4970, U2 TLI4970, U3 TLI4970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

Commit message: more layout
Parts:
- added H1, H10, H2, H3, H4: VEE, MountingHole:MountingHole_3.2mm_M3_DIN965_Pad, symbol Mechanical:MountingHole_Pad
- added H11, H12: MountingHole, MountingHole:MountingHole_3.2mm_M3, symbol Mechanical:MountingHole
- added H5: LED0-, MountingHole:MountingHole_3.2mm_M3_DIN965_Pad, symbol Mechanical:MountingHole_Pad
- added H6: LED1-, MountingHole:MountingHole_3.2mm_M3_DIN965_Pad, symbol Mechanical:MountingHole_Pad
- added H7: LED2-, MountingHole:MountingHole_3.2mm_M3_DIN965_Pad, symbol Mechanical:MountingHole_Pad
- added H8: LED3-, MountingHole:MountingHole_3.2mm_M3_DIN965_Pad, symbol Mechanical:MountingHole_Pad
- added H9: LED4-, MountingHole:MountingHole_3.2mm_M3_DIN965_Pad, symbol Mechanical:MountingHole_Pad
- added J10: TEMP_LED2, Connector_PinSocket_1.27mm:PinSocket_1x02_P1.27mm_Vertical, symbol Connector:Conn_01x02_Female
- added J11: TEMP_LED3, Connector_PinSocket_1.27mm:PinSocket_1x02_P1.27mm_Vertical, symbol Connector:Conn_01x02_Female
- added J12: TEMP_LED4, Connector_PinSocket_1.27mm:PinSocket_1x02_P1.27mm_Vertical, symbol Connector:Conn_01x02_Female
- added J13, J14: DISPLAY, Connector_PinHeader_2.54mm:PinHeader_1x12_P2.54mm_Horizontal, symbol Connector:Conn_01x12_Female
- added J15: TEMP_LED5, Connector_PinSocket_1.27mm:PinSocket_1x02_P1.27mm_Vertical, symbol Connector:Conn_01x02_Female
- added J7: POWER_12V, Connector_PinSocket_2.54mm:PinSocket_1x02_P2.54mm_Vertical, symbol Connector:Conn_01x02_Female
- added J8: TEMP_LED0, Connector_PinSocket_1.27mm:PinSocket_1x02_P1.27mm_Vertical, symbol Connector:Conn_01x02_Female
- added J9: TEMP_LED1, Connector_PinSocket_1.27mm:PinSocket_1x02_P1.27mm_Vertical, symbol Connector:Conn_01x02_Female
- added TH1, TH2, TH3, TH4, TH5, TH6: 10k, Resistor_SMD:R_0603_1608Metric_Pad1.05x0.95mm_HandSolder, symbol Device:Thermistor_NTC
- U6: footprint Display_7Segment:CA56-12EWA -> custom_lib:3461AS-1
Connections:
- net GND: now also J7.1 (Pin_1)
- net a: now also J13.1 (Pin_1); no longer XA1.D42
- net b: now also J13.10 (Pin_10); no longer XA1.D43
- net c: now also J13.3 (Pin_3); no longer XA1.D44
- net d: now also J13.5 (Pin_5); no longer XA1.D45
- net digit_pin0: now also J13.9 (Pin_9); no longer XA1.D50
- net digit_pin1: now also J13.7 (Pin_7); no longer XA1.D51
- net digit_pin2: now also J13.11 (Pin_11); no longer XA1.D52 (D52_CS2)
- net digit_pin3: now also J13.12 (Pin_12); no longer XA1.D53
- net dpx: now also J13.2 (Pin_2); no longer XA1.D49
- net e: now also J13.4 (Pin_4); no longer XA1.D46
- net f: now also J13.6 (Pin_6); no longer XA1.D47
- net g: now also J13.8 (Pin_8); no longer XA1.D48
- net +12V: now reaches XA1.VIN
- net +12V: now also J7.2 (Pin_2)
- net at U1.7 (IP+): now also H5.1
- net at U1.8 (IP-): now also H1.1
- net at U2.7 (IP+): now also H6.1
- net at U2.8 (IP-): now also H2.1
- net at U3.7 (IP+): now also H7.1
- net at U3.8 (IP-): now also H3.1
- net at U4.7 (IP+): now also H8.1
- net at U4.8 (IP-): now also H4.1
- net at U5.7 (IP+): now also H9.1
- net at U5.8 (IP-): now also H10.1
- new net: J14.1 (Pin_1), XA1.D42
- new net: J14.2 (Pin_2), XA1.D43
- new net: J14.3 (Pin_3), XA1.D44
- new net: J14.4 (Pin_4), XA1.D45
- new net: J14.5 (Pin_5), XA1.D46
- new net: J14.6 (Pin_6), XA1.D47
- new net: J14.7 (Pin_7), XA1.D48
- new net: J14.8 (Pin_8), XA1.D49
- new net: J14.9 (Pin_9), XA1.D50
- new net: J14.10 (Pin_10), XA1.D51
- new net: J14.11 (Pin_11), XA1.D52 (D52_CS2)
- new net: J14.12 (Pin_12), XA1.D53
- new net: J8.1 (Pin_1), TH1.1
- new net: J8.2 (Pin_2), TH1.2
- new net: J9.1 (Pin_1), TH2.1
- new net: J9.2 (Pin_2), TH2.2
- new net: J10.1 (Pin_1), TH3.1
- new net: J10.2 (Pin_2), TH3.2
- new net: J11.1 (Pin_1), TH4.1
- new net: J11.2 (Pin_2), TH4.2
- new net: J12.1 (Pin_1), TH5.1
- new net: J12.2 (Pin_2), TH5.2
- new net: J15.1 (Pin_1), TH6.1
- new net: J15.2 (Pin_2), TH6.2
- no-connect marks 3 -> 6
Other:
- moved on the sheet: R6, R7, R8, R9, U6, XA1

Commit message: almoscht done
Parts:
- added J16: LVHC_monitor, Connector_PinHeader_2.54mm:PinHeader_1x04_P2.54mm_Vertical, symbol Connector:Conn_01x04_Female
- J13, J14: footprint Connector_PinHeader_2.54mm:PinHeader_1x12_P2.54mm_Horizontal -> Connector_PinHeader_2.54mm:PinHeader_1x12_P2.54mm_Vertical
Connections:
- net +5V: now also XA1.5V2 (SPI_5V)
- net IL_SCALED: now also J16.2 (Pin_2)
- net I_LED_SCALED: now also J16.1 (Pin_1)
- net LED_TEMP_SCALED: now also J16.4 (Pin_4)
- net LED_VOUT: now also J16.3 (Pin_3)
- no-connect marks 6 -> 5
Changed lines of the file:
@@
 Text Label 5925 1250 1    50   ~ 0
 SCK
-NoConn ~ 6025 1250
 NoConn ~ 6125 1250
 NoConn ~ 6225 1250
@@
 F 0 "J14" H 7502 5376 50  0000 L CNN
 F 1 "DISPLAY" H 7502 5285 50  0000 L CNN
-F 2 "Connector_PinHeader_2.54mm:PinHeader_1x12_P2.54mm_Horizontal" H 7475 5400 50  0001 C CNN
+F 2 "Connector_PinHeader_2.54mm:PinHeader_1x12_P2.54mm_Vertical" H 7475 5400 50  0001 C CNN
 F 3 "~" H 7475 5400 50  0001 C CNN
 	1    7475 5400
@@
 F 0 "J13" H 2177 876 50  0000 L CNN
 F 1 "DISPLAY" H 2177 785 50  0000 L CNN
-F 2 "Connector_PinHeader_2.54mm:PinHeader_1x12_P2.54mm_Horizontal" H 2150 900 50  0001 C CNN
+F 2 "Connector_PinHeader_2.54mm:PinHeader_1x12_P2.54mm_Vertical" H 2150 900 50  0001 C CNN
 F 3 "~" H 2150 900 50  0001 C CNN
 	1    2150 900
@@
 Wire Wire Line
 	2800 5525 3100 5525
+$Comp
+L power:+5V #PWR0129
+U 1 1 605489F4
+P 6025 1250
+F 0 "#PWR0129" H 6025 1100 50  0001 C CNN
+F 1 "+5V" H 6040 1423 50  0000 C CNN
+F 2 "" H 6025 1250 50  0001 C CNN
+F 3 "" H 6025 1250 50  0001 C CNN
+	1    6025 1250
+	1    0    0    -1
+$EndComp
+$Comp
+L Connector:Conn_01x04_Female J16
+U 1 1 6054A274
+P 3550 6100
+F 0 "J16" H 3577 6076 50  0000 L CNN
+F 1 "LVHC_monitor" H 3577 5985 50  0000 L CNN
+F 2 "Connector_PinHeader_2.54mm:PinHeader_1x04_P2.54mm_Vertical" H 3550 6100 50  0001 C CNN
+F 3 "~" H 3550 6100 50  0001 C CNN
+	1    3550 6100
+	1    0    0    -1
+$EndComp
+Text Label 3350 6000 2    50   ~ 0
+I_LED_SCALED
+Text Label 3350 6100 2    50   ~ 0
+IL_SCALED
+Text Label 3350 6200 2    50   ~ 0
+LED_VOUT
+Text Label 3350 6300 2    50   ~ 0
+LED_TEMP_SCALED
 $EndSCHEMATC

Commit message: with buttons
Parts:
- added J17: POTI, Connector_PinHeader_2.54mm:PinHeader_1x03_P2.54mm_Vertical, symbol Connector:Conn_01x03_Female
- added J18: BUTTON0, Connector_PinSocket_2.54mm:PinSocket_1x02_P2.54mm_Vertical, symbol Connector:Conn_01x02_Female
- added J19: BUTTON1, Connector_PinSocket_2.54mm:PinSocket_1x02_P2.54mm_Vertical, symbol Connector:Conn_01x02_Female
- added J20: BUTTON2, Connector_PinSocket_2.54mm:PinSocket_1x02_P2.54mm_Vertical, symbol Connector:Conn_01x02_Female
- added J21: KILL0, Connector_PinSocket_2.54mm:PinSocket_1x02_P2.54mm_Vertical, symbol Connector:Conn_01x02_Female
- added J22: KILL1, Connector_PinSocket_2.54mm:PinSocket_1x02_P2.54mm_Vertical, symbol Connector:Conn_01x02_Female
Connections:
- net +3V3: now also J17.2 (Pin_2)
- net GND: now also J17.1 (Pin_1), J18.1 (Pin_1), J19.1 (Pin_1), J20.1 (Pin_1), J21.1 (Pin_1), J22.1 (Pin_1)
- net POTI: now reaches XA1.A9
- net POTI: now also J17.3 (Pin_3)
- net BUTTON2: now reaches XA1.D39
- net BUTTON2: now also J20.2 (Pin_2)
- net BUTTON1: now reaches XA1.D40
- net BUTTON1: now also J19.2 (Pin_2)
- net BUTTON0: now reaches XA1.D41
- net BUTTON0: now also J18.2 (Pin_2)
- net LED_CONTROL renamed KILL0
- net KILL0: now also J21.2 (Pin_2), J22.2 (Pin_2)
Changed lines of the file:
@@
 EESchema Schematic File Version 4
+LIBS:uven-mainboard-cache
 EELAYER 26 0
 EELAYER END
@@
 Text Label 7275 1700 0    50   ~ 0
 LED_CONTROL
-Text Label 9350 1250 2    50   ~ 0
+Text Label 9050 1250 2    50   ~ 0
 LED_CONTROL
 $Comp
@@
 Text Label 3350 6300 2    50   ~ 0
 LED_TEMP_SCALED
+$Comp
+L Connector:Conn_01x03_Female J17
+U 1 1 60512F65
+P 4675 6800
+F 0 "J17" H 4702 6826 50  0000 L CNN
+F 1 "POTI" H 4702 6735 50  0000 L CNN
+F 2 "Connector_PinHeader_2.54mm:PinHeader_1x03_P2.54mm_Vertical" H 4675 6800 50  0001 C CNN
+F 3 "~" H 4675 6800 50  0001 C CNN
+	1    4675 6800
+	1    0    0    -1
+$EndComp
+$Comp
+L power:+3.3V #PWR0130
+U 1 1 605131C7
+P 4475 6800
+F 0 "#PWR0130" H 4475 6650 50  0001 C CNN
+F 1 "+3.3V" V 4490 6928 50  0000 L CNN
+F 2 "" H 4475 6800 50  0001 C CNN
+F 3 "" H 4475 6800 50  0001 C CNN
+	1    4475 6800
+	0    -1   -1   0
+$EndComp
+$Comp
+L power:GND #PWR0131
+U 1 1 60513246
+P 4475 6700
+F 0 "#PWR0131" H 4475 6450 50  0001 C CNN
+F 1 "GND" V 4480 6572 50  0000 R CNN
+F 2 "" H 4475 6700 50  0001 C CNN
+F 3 "" H 4475 6700 50  0001 C CNN
+	1    4475 6700
+	0    1    1    0
+$EndComp
+Text Label 4475 6900 2    50   ~ 0
+POTI
+Text Label 4675 4300 2    50   ~ 0
+POTI
+$Comp
+L Connector:Conn_01x02_Female J18
+U 1 1 60513E84
+P 1700 6425
+F 0 "J18" H 1594 6100 50  0000 C CNN
+F 1 "BUTTON0" H 1594 6191 50  0000 C CNN
+F 2 "Connector_PinSocket_2.54mm:PinSocket_1x02_P2.54mm_Vertical" H 1700 6425 50  0001 C CNN
+F 3 "~" H 1700 6425 50  0001 C CNN
+	1    1700 6425
+	-1   0    0    1
+$EndComp
+Text Label 1900 6325 0    50   ~ 0
+BUTTON0
+$Comp
+L power:GND #PWR0132
+U 1 1 605141F3
+P 1900 6425
+F 0 "#PWR0132" H 1900 6175 50  0001 C CNN
+F 1 "GND" V 1905 6297 50  0000 R CNN
+F 2 "" H 1900 6425 50  0001 C CNN
+F 3 "" H 1900 6425 50  0001 C CNN
+	1    1900 6425
+	0    -1   -1   0
+$EndComp
+$Comp
+L Connector:Conn_01x02_Female J19
+U 1 1 605143DC
+P 1700 6900
+F 0 "J19" H 1594 6575 50  0000 C CNN
+F 1 "BUTTON1" H 1594 6666 50  0000 C CNN
+F 2 "Connector_PinSocket_2.54mm:PinSocket_1x02_P2.54mm_Vertical" H 1700 6900 50  0001 C CNN
+F 3 "~" H 1700 6900 50  0001 C CNN
+	1    1700 6900
+	-1   0    0    1
+$EndComp
+Text Label 1900 6800 0    50   ~ 0
+BUTTON1
+$Comp
+L power:GND #PWR0133
+U 1 1 605143E4
+P 1900 6900
+F 0 "#PWR0133" H 1900 6650 50  0001 C CNN
+F 1 "GND" V 1905 6772 50  0000 R CNN
+F 2 "" H 1900 6900 50  0001 C CNN
+F 3 "" H 1900 6900 50  0001 C CNN
+	1    1900 6900
+	0    -1   -1   0
+$EndComp
+$Comp
+L Connector:Conn_01x02_Female J20
+U 1 1 60515B18
+P 1700 7350
+F 0 "J20" H 1594 7025 50  0000 C CNN
+F 1 "BUTTON2" H 1594 7116 50  0000 C CNN
+F 2 "Connector_PinSocket_2.54mm:PinSocket_1x02_P2.54mm_Vertical" H 1700 7350 50  0001 C CNN
+F 3 "~" H 1700 7350 50  0001 C CNN
+	1    1700 7350
+	-1   0    0    1
+$EndComp
+Text Label 1900 7250 0    50   ~ 0
+BUTTON2
+$Comp
+L power:GND #PWR0134
+U 1 1 60515B20
+P 1900 7350
+F 0 "#PWR0134" H 1900 7100 50  0001 C CNN
+F 1 "GND" V 1905 7222 50  0000 R CNN
+F 2 "" H 1900 7350 50  0001 C CNN
+F 3 "" H 1900 7350 50  0001 C CNN
+	1    1900 7350
+	0    -1   -1   0
+$EndComp
+Text Label 7275 4800 0    50   ~ 0
+BUTTON0
+Text Label 7275 4700 0    50   ~ 0
+BUTTON1
+Text Label 7275 4600 0    50   ~ 0
+BUTTON2
+$Comp
+L Connector:Conn_01x02_Female J21
+U 1 1 605179F8
+P 2750 6900
+F 0 "J21" H 2644 6575 50  0000 C CNN
+F 1 "KILL0" H 2644 6666 50  0000 C CNN
+F 2 "Connector_PinSocket_2.54mm:PinSocket_1x02_P2.54mm_Vertical" H 2750 6900 50  0001 C CNN
+F 3 "~" H 2750 6900 50  0001 C CNN
+	1    2750 6900
+	-1   0    0    1
+$EndComp
+Text Label 2950 6800 0    50   ~ 0
+KILL0
+$Comp
+L power:GND #PWR0135
+U 1 1 60517A00
+P 2950 6900
+F 0 "#PWR0135" H 2950 6650 50  0001 C CNN
+F 1 "GND" V 2955 6772 50  0000 R CNN
+F 2 "" H 2950 6900 50  0001 C CNN
+F 3 "" H 2950 6900 50  0001 C CNN
+	1    2950 6900
+	0    -1   -1   0
+$EndComp
+$Comp
+L Connector:Conn_01x02_Female J22
+U 1 1 605189B4
+P 2750 7325
+F 0 "J22" H 2644 7000 50  0000 C CNN
+F 1 "KILL1" H 2644 7091 50  0000 C CNN
+F 2 "Connector_PinSocket_2.54mm:PinSocket_1x02_P2.54mm_Vertical" H 2750 7325 50  0001 C CNN
+F 3 "~" H 2750 7325 50  0001 C CNN
+	1    2750 7325
+	-1   0    0    1
+$EndComp
+Text Label 2950 7225 0    50   ~ 0
+KILL1
+$Comp
+L power:GND #PWR0136
+U 1 1 605189BC
+P 2950 7325
+F 0 "#PWR0136" H 2950 7075 50  0001 C CNN
+F 1 "GND" V 2955 7197 50  0000 R CNN
+F 2 "" H 2950 7325 50  0001 C CNN
+F 3 "" H 2950 7325 50  0001 C CNN
+	1    2950 7325
+	0    -1   -1   0
+$EndComp
+Wire Wire Line
+	9350 1250 9050 1250
+Text Label 9050 1375 2    50   ~ 0
+KILL0
+Text Label 9050 1475 2    50   ~ 0
+KILL1
+Wire Wire Line
+	9350 1375 9350 1250
+Wire Wire Line
+	9050 1375 9350 1375
+Connection ~ 9350 1250
+Wire Wire Line
+	9050 1475 9350 1475
+Wire Wire Line
+	9350 1475 9350 1375
+Connection ~ 9350 1375
 $EndSCHEMATC
