File: hardware/uven-mainboard/uven-mainboard.kicad_pcb (KiCad board)
At the start: 2 copper layers, 29 parts, among them J1 TEMP_LED0, J2 TEMP_LED1, J3 TEMP_LED2, J4 TEMP_LED3, J5 TEMP_LED4, J6 LED_CONTROL, Q1 2N7002, U1 TLI4970, U2 TLI4970, U3 TLI4970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

Commit message: more layout
Parts:
- added H1: VEE, MountingHole:MountingHole_3.2mm_M3_DIN965_Pad, F.Cu at (198.0, 51.0)
- added H10: VEE, MountingHole:MountingHole_3.2mm_M3_DIN965_Pad, F.Cu at (114.0, 51.0)
- added H11: MountingHole, MountingHole:MountingHole_3.2mm_M3, F.Cu at (223.5, 79.0)
- added H12: MountingHole, MountingHole:MountingHole_3.2mm_M3, F.Cu at (223.5, 119.0)
- added H2: VEE, MountingHole:MountingHole_3.2mm_M3_DIN965_Pad, F.Cu at (177.0, 51.0)
- added H3: VEE, MountingHole:MountingHole_3.2mm_M3_DIN965_Pad, F.Cu at (156.0, 51.0)
- added H4: VEE, MountingHole:MountingHole_3.2mm_M3_DIN965_Pad, F.Cu at (135.0, 51.0)
- added H5: LED0-, MountingHole:MountingHole_3.2mm_M3_DIN965_Pad, F.Cu at (206.0, 51.0)
- added H6: LED1-, MountingHole:MountingHole_3.2mm_M3_DIN965_Pad, F.Cu at (185.0, 51.0)
- added H7: LED2-, MountingHole:MountingHole_3.2mm_M3_DIN965_Pad, F.Cu at (164.0, 51.0)
- added H8: LED3-, MountingHole:MountingHole_3.2mm_M3_DIN965_Pad, F.Cu at (143.0, 51.0)
- added H9: LED4-, MountingHole:MountingHole_3.2mm_M3_DIN965_Pad, F.Cu at (122.0, 51.0)
- added J10: TEMP_LED2, Connector_PinSocket_1.27mm:PinSocket_1x02_P1.27mm_Vertical, F.Cu at (250.0, 101.0)
- added J11: TEMP_LED3, Connector_PinSocket_1.27mm:PinSocket_1x02_P1.27mm_Vertical, F.Cu at (250.0, 95.0)
- added J12: TEMP_LED4, Connector_PinSocket_1.27mm:PinSocket_1x02_P1.27mm_Vertical, F.Cu at (250.0, 89.0)
- added J13: DISPLAY, Connector_PinHeader_2.54mm:PinHeader_1x12_P2.54mm_Horizontal, B.Cu at (230.5, 85.5)
- added J14: DISPLAY, Connector_PinHeader_2.54mm:PinHeader_1x12_P2.54mm_Horizontal, F.Cu at (190.0, 86.0)
- added J15: TEMP_LED5, Connector_PinSocket_1.27mm:PinSocket_1x02_P1.27mm_Vertical, F.Cu at (250.1, 82.7)
- added J7: POWER_12V, Connector_PinSocket_2.54mm:PinSocket_1x02_P2.54mm_Vertical, F.Cu at (153.0, 117.0)
- added J8: TEMP_LED0, Connector_PinSocket_1.27mm:PinSocket_1x02_P1.27mm_Vertical, F.Cu at (250.0, 113.0)
- added J9: TEMP_LED1, Connector_PinSocket_1.27mm:PinSocket_1x02_P1.27mm_Vertical, F.Cu at (250.0, 107.0)
- added TH1: 10k, Resistor_SMD:R_0603_1608Metric_Pad1.05x0.95mm_HandSolder, F.Cu at (253.0, 112.5)
- added TH2: 10k, Resistor_SMD:R_0603_1608Metric_Pad1.05x0.95mm_HandSolder, F.Cu at (253.0, 106.5)
- added TH3: 10k, Resistor_SMD:R_0603_1608Metric_Pad1.05x0.95mm_HandSolder, F.Cu at (253.0, 100.5)
- added TH4: 10k, Resistor_SMD:R_0603_1608Metric_Pad1.05x0.95mm_HandSolder, F.Cu at (253.0, 94.5)
- added TH5: 10k, Resistor_SMD:R_0603_1608Metric_Pad1.05x0.95mm_HandSolder, F.Cu at (253.0, 88.5)
- added TH6: 10k, Resistor_SMD:R_0603_1608Metric_Pad1.05x0.95mm_HandSolder, F.Cu at (253.0, 82.0)
- R6, R7, R8, R9: moved to B.Cu
- U6: footprint Display_7Segment:CA56-12EWA -> custom_lib:3461AS-1
- moved C5 130.6 mm to (113.0, 64.9), turned to 90 degrees
- moved C4 111.4 mm to (134.0, 65.0), turned to 90 degrees
- moved R1 95.0 mm to (149.0, 109.0), turned to 270 degrees
- moved C3 93.9 mm to (155.0, 65.0), turned to 90 degrees
- moved J6 93.4 mm to (161.0, 77.0)
- moved R10 91.6 mm to (157.0, 79.0)
- moved R2 87.5 mm to (153.0, 109.0), turned to 270 degrees
- moved R4 86.3 mm to (161.0, 109.0), turned to 270 degrees
- moved J1 85.0 mm to (149.0, 105.0), turned to 180 degrees
- moved J2 84.7 mm to (153.0, 105.0), turned to 180 degrees
- moved J3 84.3 mm to (157.0, 105.0), turned to 180 degrees
- moved J4 83.9 mm to (161.0, 105.0), turned to 180 degrees
- moved J5 83.5 mm to (165.0, 105.0), turned to 180 degrees
- moved R3 83.4 mm to (157.0, 109.0), turned to 270 degrees
- moved R5 78.8 mm to (165.0, 109.0), turned to 270 degrees
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Connections:
- XA1 pad D42: /a -> Net-(J14-Pad1)
- XA1 pad D43: /b -> Net-(J14-Pad2)
- XA1 pad D44: /c -> Net-(J14-Pad3)
- XA1 pad D45: /d -> Net-(J14-Pad4)
- XA1 pad D46: /e -> Net-(J14-Pad5)
- XA1 pad D47: /f -> Net-(J14-Pad6)
- XA1 pad D48: /g -> Net-(J14-Pad7)
- XA1 pad D49: /dpx -> Net-(J14-Pad8)
- XA1 pad D50: /digit_pin0 -> Net-(J14-Pad9)
- XA1 pad D51: /digit_pin1 -> Net-(J14-Pad10)
- XA1 pad D52: /digit_pin2 -> Net-(J14-Pad11)
- XA1 pad D53: /digit_pin3 -> Net-(J14-Pad12)
- XA1 pad VIN: Net-(XA1-PadVIN) -> +12V
Routing:
- net /dpx: track 0.00 -> 24.8 mm
- net /c: track 0.00 -> 22.3 mm, vias 0 -> 1
- net /digit_pin0: track 0.00 -> 20.1 mm
- net /g: track 0.00 -> 15.0 mm, vias 0 -> 1
- net /e: track 0.00 -> 14.4 mm
- net /d: track 0.00 -> 14.4 mm
- net /a: track 0.00 -> 12.3 mm
- net /digit_pin1: track 0.00 -> 9.40 mm
- net /digit_pin2: track 0.00 -> 8.45 mm
- net /digit_pin3: track 0.00 -> 7.84 mm
- net Net-(R9-Pad2): track 0.00 -> 7.05 mm
- net Net-(R8-Pad2): track 0.00 -> 6.86 mm, vias 0 -> 1
- net /b: track 0.00 -> 4.54 mm
- net Net-(R7-Pad2): track 0.00 -> 3.62 mm
- net /f: track 0.00 -> 3.51 mm
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
Commit message: almoscht done
Parts:
- added J16: LVHC_monitor, Connector_PinHeader_2.54mm:PinHeader_1x04_P2.54mm_Vertical, F.Cu at (174.5, 109.0)
- J13, J14: footprint Connector_PinHeader_2.54mm:PinHeader_1x12_P2.54mm_Horizontal -> Connector_PinHeader_2.54mm:PinHeader_1x12_P2.54mm_Vertical
- moved TH3 56.3 mm to (232.6, 48.0)
- moved J10 56.1 mm to (230.0, 48.6)
- moved TH2 53.5 mm to (232.6, 57.0)
- moved J9 53.3 mm to (230.0, 57.6)
- moved TH1 50.8 mm to (232.6, 66.0)
- moved J8 50.5 mm to (230.0, 66.6)
- moved TH6 45.6 mm to (222.6, 48.0)
- moved J15 45.4 mm to (220.0, 48.6)
- moved TH5 43.8 mm to (222.6, 57.0)
- moved J12 43.4 mm to (220.0, 57.6)
- moved TH4 41.7 mm to (222.6, 66.0)
- moved J11 41.3 mm to (220.0, 66.6)
- moved H11 4.74 mm to (228.0, 80.5)
- moved H12 4.74 mm to (228.0, 120.5)
- moved J13 4.74 mm to (235.0, 87.0)
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Connections:
- XA1 pad 5V2: Net-(XA1-Pad5V2) -> +5V
Routing:
- net +3V3: track 0.00 -> 220.9 mm, vias 0 -> 5
- net /SCK: track 0.00 -> 179.2 mm, vias 0 -> 5
- net /MISO: track 0.00 -> 170.4 mm, vias 0 -> 5
- net /OCD_LED0: track 0.00 -> 57.1 mm
- net /CS_LED0: track 0.00 -> 42.6 mm, vias 0 -> 1
- net /CS_LED4: track 0.00 -> 40.4 mm, vias 0 -> 1
- net /OCD_LED1: track 0.00 -> 40.0 mm
- net /CS_LED1: track 0.00 -> 30.8 mm, vias 0 -> 1
- net +5V: track 0.00 -> 27.0 mm
- net /CS_LED3: track 0.00 -> 24.4 mm, vias 0 -> 1
- net /OCD_LED4: track 0.00 -> 24.2 mm
- net /TEMP_LED0: track 0.00 -> 23.5 mm
- net /TEMP_LED1: track 0.00 -> 22.5 mm
- net Net-(J14-Pad2): track 0.00 -> 22.3 mm
- net /OCD_LED2: track 0.00 -> 21.8 mm
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- added copper zone on B.Cu, net GND
- added copper zone on F.Cu, net GND
- added copper zone on F.Cu, net Net-(H1-Pad1)
- added copper zone on F.Cu, net Net-(H10-Pad1)
- added copper zone on F.Cu, net Net-(H2-Pad1)
- added copper zone on F.Cu, net Net-(H3-Pad1)
- added copper zone on F.Cu, net Net-(H4-Pad1)
- added copper zone on F.Cu, net Net-(H5-Pad1)
- added copper zone on F.Cu, net Net-(H6-Pad1)
- added copper zone on F.Cu, net Net-(H7-Pad1)
- added copper zone on F.Cu, net Net-(H8-Pad1)
- added copper zone on F.Cu, net Net-(H9-Pad1)
Other:
- board outline added: 128 x 79 mm
- board text added: "+"
- board text added: "-"
- board text added: "0"
- board text added: "1"
- board text added: "100n"
- board text added: "10k"
- board text added: "12V"
- board text added: "2"
- board text added: "2N7002"
- board text added: "3"
- board text added: "330"
- board text added: "4"
- board text added: "5V"
- board text added: "D42"
- board text added: "D43"
- board text added: "D44"
- board text added: "D45"
- board text added: "D46"
- board text added: "D47"
- board text added: "D48"
- board text added: "D49"
- board text added: "D50"
- board text added: "D51"
- board text added: "D52"
- board text added: "D53"
- board text added: "GND"
- board text added: "IL_LED"
- board text added: "I_LED"
- board text added: "LED"
- board text added: "LED_TEMP"
- board text added: "LED_VOUT"
- board text added: "MISO"
- board text added: "MOSI"
- board text added: "SCK"
- board text added: "TLI4970"
- board text added: "a"
- board text added: "b"
- board text added: "c"
- board text added: "d"
- board text added: "dpx"
- board text added: "e"
- board text added: "f"
- board text added: "g"

Commit message: with buttons
Parts:
- added J17: POTI, Connector_PinHeader_2.54mm:PinHeader_1x03_P2.54mm_Vertical, F.Cu at (159.0, 97.0)
- added J18: BUTTON0, Connector_PinSocket_2.54mm:PinSocket_1x02_P2.54mm_Vertical, F.Cu at (194.5, 77.0)
- added J19: BUTTON1, Connector_PinSocket_2.54mm:PinSocket_1x02_P2.54mm_Vertical, F.Cu at (189.5, 77.0)
- added J20: BUTTON2, Connector_PinSocket_2.54mm:PinSocket_1x02_P2.54mm_Vertical, F.Cu at (199.5, 77.0)
- added J21: KILL0, Connector_PinSocket_2.54mm:PinSocket_1x02_P2.54mm_Vertical, F.Cu at (176.8, 77.3)
- added J22: KILL1, Connector_PinSocket_2.54mm:PinSocket_1x02_P2.54mm_Vertical, F.Cu at (182.5, 77.3)
Connections:
- net /LED_CONTROL renamed /KILL0
- XA1 pad A9: Net-(XA1-PadA9) -> /POTI
- XA1 pad D39: Net-(XA1-PadD39) -> /BUTTON2
- XA1 pad D40: Net-(XA1-PadD40) -> /BUTTON1
- XA1 pad D41: Net-(XA1-PadD41) -> /BUTTON0
Routing:
- net /POTI: track 0.00 -> 39.0 mm
- net /BUTTON1: track 0.00 -> 25.4 mm
- net /BUTTON0: track 0.00 -> 24.2 mm
- net /BUTTON2: track 0.00 -> 18.7 mm
- net /KILL0: track 9.05 -> 23.8 mm
- net +3V3: track 220.9 -> 233.8 mm
Other:
- board text added: "3.3V"
- board text added: "BUTTON0"
- board text added: "BUTTON1"
- board text added: "BUTTON2"
- board text added: "KILL0"
- board text added: "KILL1"
- board text added: "POTI"

Commit message: done and ordered
Routing:
- net Net-(H9-Pad1): vias 0 -> 51
- net Net-(H8-Pad1): vias 0 -> 45
- net Net-(H7-Pad1): vias 0 -> 44
- net Net-(H6-Pad1): vias 0 -> 44
- net Net-(H5-Pad1): vias 0 -> 43
- net Net-(H4-Pad1): vias 0 -> 49
- net Net-(H3-Pad1): vias 0 -> 49
- net Net-(H2-Pad1): vias 0 -> 49
- net Net-(H10-Pad1): vias 0 -> 49
- net Net-(H1-Pad1): vias 0 -> 49
- added copper zone on B.Cu, net Net-(H1-Pad1)
- added copper zone on B.Cu, net Net-(H10-Pad1)
- added copper zone on B.Cu, net Net-(H2-Pad1)
- added copper zone on B.Cu, net Net-(H3-Pad1)
- added copper zone on B.Cu, net Net-(H4-Pad1)
- added copper zone on B.Cu, net Net-(H5-Pad1)
- added copper zone on B.Cu, net Net-(H6-Pad1)
- added copper zone on B.Cu, net Net-(H7-Pad1)
- added copper zone on B.Cu, net Net-(H8-Pad1)
- added copper zone on B.Cu, net Net-(H9-Pad1)
Other:
- rule pad_to_mask_clearance: 0.051 -> 0

Commit message: with draft uven 2d
Other:
- net class Default removed
