File: hardware/MTSM340UV2-F5120S-current-driver/LM3407-current-controller.sch (KiCad schematic (older format))
At the start: 8 parts, among them U1 LM3407MY

Commit message: layout almost done
Parts:
- L2: footprint Inductor_SMD:L_1210_3225Metric_Pad1.42x2.65mm_HandSolder -> custom_lib:LQH3NPN
Changed lines of the file:
@@
 AR Path="/61CCE2C8/61CC7CF7" Ref="#PWR0269"  Part="1"
 AR Path="/61CCE2CE/61CC7CF7" Ref="#PWR0276"  Part="1"
-F 0 "#PWR0108" H 5150 2700 50  0001 C CNN
+F 0 "#PWR0276" H 5150 2700 50  0001 C CNN
 F 1 "GND" V 5155 2822 50  0000 R CNN
 F 2 "" H 5150 2950 50  0001 C CNN
@@
 AR Path="/61CCE2C8/61CC7D14" Ref="#PWR0270"  Part="1"
 AR Path="/61CCE2CE/61CC7D14" Ref="#PWR0277"  Part="1"
-F 0 "#PWR0109" H 6600 3700 50  0001 C CNN
+F 0 "#PWR0277" H 6600 3700 50  0001 C CNN
 F 1 "GND" H 6605 3777 50  0000 C CNN
 F 2 "" H 6600 3950 50  0001 C CNN
@@
 F 0 "L2" V 5246 3856 50  0000 R CNN
 F 1 "22uH" V 5155 3856 50  0000 R CNN
-F 2 "Inductor_SMD:L_1210_3225Metric_Pad1.42x2.65mm_HandSolder" H 5200 3900 50  0001 C CNN
+F 2 "custom_lib:LQH3NPN" H 5200 3900 50  0001 C CNN
 F 3 "~" H 5200 3900 50  0001 C CNN
 	1    5200 3900
@@
 AR Path="/61CCE2C8/61CC7D33" Ref="#PWR0271"  Part="1"
 AR Path="/61CCE2CE/61CC7D33" Ref="#PWR0278"  Part="1"
-F 0 "#PWR0110" H 6800 3500 50  0001 C CNN
+F 0 "#PWR0278" H 6800 3500 50  0001 C CNN
 F 1 "+12V" V 6815 3778 50  0000 L CNN
 F 2 "" H 6800 3650 50  0001 C CNN
@@
 AR Path="/61CCE2C8/61CC7D39" Ref="#PWR0272"  Part="1"
 AR Path="/61CCE2CE/61CC7D39" Ref="#PWR0279"  Part="1"
-F 0 "#PWR0111" H 4400 3500 50  0001 C CNN
+F 0 "#PWR0279" H 4400 3500 50  0001 C CNN
 F 1 "+12V" V 4415 3778 50  0000 L CNN
 F 2 "" H 4400 3650 50  0001 C CNN
@@
 AR Path="/61CCE2C8/61CC7D51" Ref="#PWR0273"  Part="1"
 AR Path="/61CCE2CE/61CC7D51" Ref="#PWR0280"  Part="1"
-F 0 "#PWR0112" H 6500 2700 50  0001 C CNN
+F 0 "#PWR0280" H 6500 2700 50  0001 C CNN
 F 1 "GND" H 6505 2777 50  0000 C CNN
 F 2 "" H 6500 2950 50  0001 C CNN
@@
 AR Path="/61CCE2C8/61CC7D60" Ref="#PWR0274"  Part="1"
 AR Path="/61CCE2CE/61CC7D60" Ref="#PWR0281"  Part="1"
-F 0 "#PWR0113" H 4350 3100 50  0001 C CNN
+F 0 "#PWR0281" H 4350 3100 50  0001 C CNN
 F 1 "GND" V 4355 3222 50  0000 R CNN
 F 2 "" H 4350 3350 50  0001 C CNN
