File: hardware/uven-mainboard-2D/uven-mainboard.kicad_pcb (KiCad board)
At the start: 2 copper layers, 128 x 79 mm, 35 parts, among them J1 TEMP_LED0, J10 TEMP_SPECIMEN, J11 TEC1_COOLER, J12 TEC2_COOLER, J13 DISPLAY, J14 DISPLAY, J15 TEC3_COOLER, J16 MENU_BUTTON, J18 BUTTON0, J19 BUTTON1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

Commit message: pcb ordered in aisler
Parts:
- removed TH1, TH2, TH3: 10k, Resistor_SMD:R_0603_1608Metric_Pad1.05x0.95mm_HandSolder
- added H1: GND, MountingHole:MountingHole_3.2mm_M3_DIN965_Pad_TopBottom, F.Cu at (113.5, 71.5)
- added H2: 12V, MountingHole:MountingHole_3.2mm_M3_DIN965_Pad_TopBottom, F.Cu at (113.5, 106.5)
- added H3: 12V, MountingHole:MountingHole_3.2mm_M3_DIN965_Pad_TopBottom, F.Cu at (113.5, 99.5)
- added H4: GND, MountingHole:MountingHole_3.2mm_M3_DIN965_Pad_TopBottom, F.Cu at (113.5, 84.5)
- added H5: 12V, MountingHole:MountingHole_3.2mm_M3_DIN965_Pad_TopBottom, F.Cu at (113.5, 92.5)
- added H6: GND, MountingHole:MountingHole_3.2mm_M3_DIN965_Pad_TopBottom, F.Cu at (113.5, 78.0)
- added U1: BTS3011, custom_lib:BTS3011, F.Cu at (136.7, 91.2)
- added U2: BTS3011, custom_lib:BTS3011, F.Cu at (136.7, 101.5)
- added U3: BTS3011, custom_lib:BTS3011, F.Cu at (136.7, 81.0)
- J10: value TEMP_SPECIMEN -> LED1_CONTROL; footprint Connector_PinSocket_1.27mm:PinSocket_1x02_P1.27mm_Vertical -> Connector_PinHeader_2.54mm:PinHeader_1x05_P2.54mm_Vertical
- J8: value TEMP_LED0 -> ST7789_ISP_DISPLAY; footprint Connector_PinSocket_1.27mm:PinSocket_1x02_P1.27mm_Vertical -> Connector_PinHeader_2.54mm:PinHeader_1x07_P2.54mm_Vertical
- J9: value TEMP_LED1 -> LED0_CONTROL; footprint Connector_PinSocket_1.27mm:PinSocket_1x02_P1.27mm_Vertical -> Connector_PinHeader_2.54mm:PinHeader_1x05_P2.54mm_Vertical
- moved J10 68.9 mm to (167.5, 77.5), turned to 0 degrees
- moved J9 61.8 mm to (171.5, 77.5), turned to 0 degrees
- moved J16 58.5 mm to (183.0, 105.9)
- moved J8 50.8 mm to (183.0, 86.0), turned to 0 degrees
- moved J12 26.3 mm to (122.8, 108.5), turned to -90 degrees
- moved J6 20.5 mm to (122.8, 89.0), turned to -90 degrees
- moved J15 18.6 mm to (122.8, 102.0), turned to -90 degrees
- moved J5 17.2 mm to (122.8, 76.0), turned to -90 degrees
- moved J11 11.4 mm to (122.8, 95.5), turned to -90 degrees
- moved J4 10.7 mm to (122.8, 82.5), turned to -90 degrees
Connections:
- net /MISO renamed /SPI_MISO
- J10 pad 1: Net-(J10-Pad1) -> GND
- J10 pad 2: Net-(J10-Pad2) -> +3V3
- J22 pad 2: /KILL_0 -> /KILL0
- J3 pad 1: /TEMP_SPECISMEN -> /TEMP_SPECIMEN
- J4 pad 1: GND -> Net-(U1-Pad6)
- J4 pad 2: Net-(J4-Pad2) -> +12V
- J5 pad 1: GND -> Net-(U3-Pad6)
- J5 pad 2: Net-(J5-Pad2) -> +12V
- J8 pad 1: Net-(J8-Pad1) -> GND
- J8 pad 2: Net-(J8-Pad2) -> +3V3
- J9 pad 1: Net-(J9-Pad1) -> GND
- J9 pad 2: Net-(J9-Pad2) -> +3V3
- R3 pad 1: /TEMP_SPECISMEN -> /TEMP_SPECIMEN
- XA1 pad D11: unconnected-(XA1-PadD11) -> /MENU_BUTTON
- XA1 pad D12: unconnected-(XA1-PadD12) -> /MENU_DT
- XA1 pad D13: unconnected-(XA1-PadD13) -> /MENU_CLK
- XA1 pad D14: unconnected-(XA1-PadD14) -> /LED0_ON/OFF
- XA1 pad D15: unconnected-(XA1-PadD15) -> /LED1_ON/OFF
- XA1 pad D2: /TEC_LED0_IN -> /TEC_COOLER_IN
- XA1 pad D20: unconnected-(XA1-PadD20) -> /LED0_I2C_SDA
- XA1 pad D21: unconnected-(XA1-PadD21) -> /LED0_I2C_SCL
- XA1 pad D28: unconnected-(XA1-PadD28) -> /KILL0
- XA1 pad D35: unconnected-(XA1-PadD35) -> /ISP_RES
- XA1 pad D36: unconnected-(XA1-PadD36) -> /ISP_DC
- XA1 pad D37: unconnected-(XA1-PadD37) -> /ISP_BLK
- XA1 pad D38: /KILL0 -> unconnected-(XA1-PadD38)
- XA1 pad D4: /TEC_COOLER_IN -> /TEC_LED0_IN
- XA1 pad D5: /TEC_LED0_STATUS -> /TEC_COOLER_STATUS
- XA1 pad D7: /TEC_COOLER_STATUS -> /TEC_LED0_STATUS
- XA1 pad MOSI: /MOSI -> /SPI_MOSI
- XA1 pad SCK: /SCK -> /SPI_SCK
- XA1 pad SCL1: unconnected-(XA1-PadSCL1) -> /LED1_I2C_SCL
- XA1 pad SDA1: unconnected-(XA1-PadSDA1) -> /LED1_I2C_SDA
Routing:
- net +12V: track 3.53 -> 144.5 mm
- net +3V3: track 20.8 -> 152.2 mm, vias 0 -> 3
- net /LED1_I2C_SCL: track 0.00 -> 69.5 mm
- net /LED1_I2C_SDA: track 0.00 -> 68.4 mm
- net Net-(J11-Pad1): track 0.00 -> 66.4 mm, vias 0 -> 36
- net /MENU_CLK: track 0.00 -> 62.2 mm
- net /MENU_DT: track 0.00 -> 58.6 mm
- net /MENU_BUTTON: track 0.00 -> 55.0 mm
- net /TEC_COOLER_IN: track 0.00 -> 42.9 mm
- net /LED0_I2C_SCL: track 0.00 -> 36.8 mm
- net /TEC_COOLER_STATUS: track 0.00 -> 36.3 mm, vias 0 -> 1
- net /LED0_I2C_SDA: track 0.00 -> 36.0 mm
- net /ISP_BLK: track 0.00 -> 32.7 mm
- net /TEC_LED1_IN: track 0.00 -> 31.7 mm
- net /LED1_ON/OFF: track 0.00 -> 27.3 mm
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Other:
- board size 128 x 79 mm -> 128 x 57.5 mm
- board text added: "3.3V"
- board text added: "BLK"
- board text added: "BUT"
- board text added: "CLK"
- board text added: "DC"
- board text added: "DT"
- board text added: "LED0"
- board text added: "LED1"
- board text added: "MOSI"
- board text added: "ON/OFF"
- board text added: "RES"
- board text added: "SCK"
- board text added: "SCL"
- board text added: "SDA"
