File: hardware/poti_hack/poti_hack.kicad_pcb (KiCad board)
At the start: 2 copper layers, 12.5 x 11.6 mm, 6 parts, among them J1 POTI_i2c, J2 POTI, U1 MCP4018-xxxxLT

Commit message: v1 ordered on aisler
Other:
- board text added: "poti_hack_v1"

Commit message: led control draft
Other:
- net class Default removed
