File: hardware/uven2-mk2-mainboard/led_driver.kicad_sch (KiCad schematic)
At the start: 5 parts, among them J1 LED, Q1 QM6006D

Commit message: with current limiting switch
Parts:
- removed R2: 220mOhm, Resistor_SMD:R_2512_6332Metric_Pad1.40x3.35mm_HandSolder, symbol Device:R
- added C7: 100n, Capacitor_SMD:C_0603_1608Metric_Pad1.08x0.95mm_HandSolder, symbol Device:C
- added C8: 220n, Capacitor_SMD:C_0603_1608Metric_Pad1.08x0.95mm_HandSolder, symbol Device:C
- added C9: 4.7u, Capacitor_SMD:C_0603_1608Metric_Pad1.08x0.95mm_HandSolder, symbol Device:C
- added J3: LED, Connector_PinHeader_2.54mm:PinHeader_1x02_P2.54mm_Vertical, symbol Connector:Conn_01x02_Female
- added Q2: QM6006D, Package_TO_SOT_SMD:TO-252-2, symbol Transistor_FET:QM6006D
- added R3: 1k, Resistor_SMD:R_0603_1608Metric_Pad0.98x0.95mm_HandSolder, symbol Device:R
- added R4, R5: 10k, Resistor_SMD:R_0603_1608Metric_Pad0.98x0.95mm_HandSolder, symbol Device:R
- added U4: TPS2HB50BQPWPRQ1, custom_lib:SOP65P640X120-17N, symbol TPS2HB50BQPWPRQ1:TPS2HB50BQPWPRQ1
Connections:
- net SHUNT_LED0 is gone; now on net GND: Q1.3 (S)
- net +24V: now also C8.2, C9.2, R4.1, R5.1, U4.17 (VBB); no longer J1.1 (Pin_1)
- net GND: now also C7.1, C8.1, C9.1, Q2.3 (S), R3.1, U4.1 (GND)
- new net: J3.2 (Pin_2), Q2.2 (D)
- new net: R4.2, U4.5 (ILIM1)
- new net: R5.2, U4.12 (ILIM2)
- new net GATE_LED1: C7.2, Q2.1 (G), R3.2
- new net LED0: U4.6 (VOUT1), U4.7 (VOUT1), U4.8 (VOUT1)
- new net LED1: U4.10 (VOUT2), U4.11 (VOUT2), U4.9 (VOUT2)
- new net LED_DIAG_EN: U4.16 (DIA_EN)
- new net LED_EN: U4.13 (EN2), U4.4 (EN1)
- new net LED_LATCH: U4.3 (LATCH)
- new net LED_SEL0: U4.14 (SEL1)
- new net LED_SEL1: U4.15 (SEL2)
- new net LED_SENS: U4.2 (SNS)
Other:
- note added: "Rsens shared between all switches"
- moved on the sheet: C5, J1, Q1, R1

Commit message: with wago connector
Parts:
- removed J1, J3: LED, Connector_PinHeader_2.54mm:PinHeader_1x02_P2.54mm_Vertical, symbol Connector:Conn_01x02_Female
- added R34, R35: 10k, Resistor_SMD:R_0603_1608Metric_Pad1.05x0.95mm_HandSolder, symbol uven-mainboard-rescue:R-Device
Connections:
- net LED0-: now reaches Q1.2 (D)
- net LED1-: now reaches Q2.2 (D)
- net LED0 renamed LED0+
- net LED1 renamed LED1+
- new net +3V3: R34.2, R35.2
- new net TEMP_LED0: R34.1
- new net TEMP_LED1: R35.1
Other:
- moved on the sheet: C5, Q1, R1

Commit message: with different mosfet
Parts:
- removed Q1, Q2: QM6006D, Package_TO_SOT_SMD:TO-252-2, symbol Transistor_FET:QM6006D
- added U12, U13: SIDR392DP-T1-GE3, custom_lib:PowerPAK SO-8DC, symbol custom:SIDR392DP-T1-GE3
Connections:
- net GATE_LED0: now also U12.4 (G)
- net GATE_LED1: now also U13.4 (G)
- net GND: now also U12.1 (S), U12.2 (S), U12.3 (S), U13.1 (S), U13.2 (S), U13.3 (S)
- net LED0-: now also U12.5 (D)
- net LED1-: now also U13.5 (D)
Other:
- moved on the sheet: C7, R3

Commit message: schematics done
Parts:
- R34, R35: footprint Resistor_SMD:R_0603_1608Metric_Pad1.05x0.95mm_HandSolder -> Resistor_SMD:R_0603_1608Metric_Pad0.98x0.95mm_HandSolder
Changed lines of the file:
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@@
     (property "Reference" "R34" (id 0) (at 167.005 46.355 90))
     (property "Value" "10k" (id 1) (at 170.18 48.26 90))
-    (property "Footprint" "Resistor_SMD:R_0603_1608Metric_Pad1.05x0.95mm_HandSolder" (id 2) (at 170.18 46.482 90)
+    (property "Footprint" "Resistor_SMD:R_0603_1608Metric_Pad0.98x0.95mm_HandSolder" (id 2) (at 170.18 46.482 90)
       (effects (font (size 1.27 1.27)) hide)
     )
@@
     (property "Reference" "R35" (id 0) (at 167.005 51.435 90))
     (property "Value" "10k" (id 1) (at 170.18 53.34 90))
-    (property "Footprint" "Resistor_SMD:R_0603_1608Metric_Pad1.05x0.95mm_HandSolder" (id 2) (at 170.18 51.562 90)
-      (effects (font (size 1.27 1.27)) hide)
-    )
+    (property "Footprint" "Resistor_SMD:R_0603_1608Metric_Pad0.98x0.95mm_HandSolder" (id 2) (at 170.18 51.562 90)
+      (effects (font (size 1.27 1.27)) hide)
+    )

Commit message: layout almost finished
Connections:
- net +3V3 renamed +3.3V
Changed lines of the file:
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@@
+    (stroke (width 0) (type default) (color 0 0 0 0))
+  )
+  (wire (pts (xy 163.83 53.34) (xy 166.37 53.34))
     (stroke (width 0) (type default) (color 0 0 0 0))
   )
@@
   )
   (wire (pts (xy 172.72 113.03) (xy 176.53 113.03))
+    (stroke (width 0) (type default) (color 0 0 0 0))
+  )
+  (wire (pts (xy 163.83 48.26) (xy 166.37 48.26))
     (stroke (width 0) (type default) (color 0 0 0 0))
   )
@@
     (pin "1")
   )
+  (symbol (lib_id "power:+3.3V") (at 163.83 48.26 90) (unit 1)
+    (in_bom yes) (on_board yes)
+    (property "Reference" "#PWR0198" (id 0) (at 167.64 48.26 0)
+      (effects (font (size 1.27 1.27)) hide)
+    )
+    (property "Value" "+3.3V" (id 1) (at 158.75 45.72 90)
+      (effects (font (size 1.27 1.27)) (justify right))
+    )
+    (property "Footprint" "" (id 2) (at 163.83 48.26 0)
+      (effects (font (size 1.27 1.27)) hide)
+    )
+    (property "Datasheet" "" (id 3) (at 163.83 48.26 0)
+      (effects (font (size 1.27 1.27)) hide)
+    )
+    (pin "1")
+  )
   (symbol (lib_id "custom:SIDR392DP-T1-GE3") (at 123.19 66.04 0) (unit 1)
     (in_bom yes) (on_board yes)
@@
     (pin "1")
   )
-  (symbol (lib_id "uven-mainboard-rescue:+3.3V-power") (at 166.37 53.34 90) (unit 1)
-    (in_bom yes) (on_board yes)
-    (property "Reference" "#PWR0198" (id 0) (at 170.18 53.34 0)
-      (effects (font (size 1.27 1.27)) hide)
-    )
-    (property "Value" "+3.3V" (id 1) (at 163.1188 52.959 90)
-      (effects (font (size 1.27 1.27)) (justify left))
-    )
-    (property "Footprint" "" (id 2) (at 166.37 53.34 0)
-      (effects (font (size 1.27 1.27)) hide)
-    )
-    (property "Datasheet" "" (id 3) (at 166.37 53.34 0)
-      (effects (font (size 1.27 1.27)) hide)
-    )
-    (pin "1")
-  )
   (symbol (lib_id "custom:SIDR392DP-T1-GE3") (at 123.19 109.22 0) (unit 1)
     (in_bom yes) (on_board yes)
@@
     (pin "1")
     (pin "2")
-  )
-  (symbol (lib_id "uven-mainboard-rescue:+3.3V-power") (at 166.37 48.26 90) (unit 1)
-    (in_bom yes) (on_board yes)
-    (property "Reference" "#PWR0199" (id 0) (at 170.18 48.26 0)
-      (effects (font (size 1.27 1.27)) hide)
-    )
-    (property "Value" "+3.3V" (id 1) (at 163.1188 47.879 90)
-      (effects (font (size 1.27 1.27)) (justify left))
-    )
-    (property "Footprint" "" (id 2) (at 166.37 48.26 0)
-      (effects (font (size 1.27 1.27)) hide)
-    )
-    (property "Datasheet" "" (id 3) (at 166.37 48.26 0)
-      (effects (font (size 1.27 1.27)) hide)
-    )
-    (pin "1")
   )
   (symbol (lib_id "Device:R") (at 100.33 105.41 0) (unit 1)
@@
     (pin "9")
   )
+  (symbol (lib_id "power:+3.3V") (at 163.83 53.34 90) (unit 1)
+    (in_bom yes) (on_board yes)
+    (property "Reference" "#PWR0199" (id 0) (at 167.64 53.34 0)
+      (effects (font (size 1.27 1.27)) hide)
+    )
+    (property "Value" "+3.3V" (id 1) (at 158.75 50.8 90)
+      (effects (font (size 1.27 1.27)) (justify right))
+    )
+    (property "Footprint" "" (id 2) (at 163.83 53.34 0)
+      (effects (font (size 1.27 1.27)) hide)
+    )
+    (property "Datasheet" "" (id 3) (at 163.83 53.34 0)
+      (effects (font (size 1.27 1.27)) hide)
+    )
+    (pin "1")
+  )
   (symbol (lib_id "Device:R") (at 102.87 62.23 0) (unit 1)
