File: hardware/uven2-mk2-mainboard/uven2-mk2-mainboard.kicad_pcb (KiCad board)
At the start: 4 copper layers, 176.8 x 115.3 mm, 210 parts, among them J1 LEDs, J10 GND, J11 24V, J12 GND, J13 24V, J14 GND, J15 Chamber_Control, J16 USB_A, J17 PowerON/OFF, J2 1-282834-0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

Commit message: fixed 3.3V trace missing, added footage
Connections:
- R50 pad 2: +3V3 -> +3.3V
Routing:
- net +3.3V: track 211.2 -> 214.8 mm
