File: hardware/uven-pocket-main-board/uven-pocket-main-board.kicad_sch (KiCad schematic)
At the start: 39 parts, among them J1 Raspberry_Pi_2_3, J10 VDrive, J11 GND, J2 FAN, J3 TEMP_CHAMBER1, J4 TEMP_CHAMBER0, J5 1-282834-2, J6 VDrive, J7 GND, J8 VDrive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

Commit message: single led copper base + uven pocket finished
Parts:
- added D1, D2, D3: LED, LED_SMD:LED_0603_1608Metric_Pad1.05x0.95mm_HandSolder, symbol Device:LED
- added H1, H2, H3, H4: MountingHole, MountingHole:MountingHole_3.2mm_M3, symbol Mechanical:MountingHole
- added J12: 3.3V, Connector_PinSocket_2.54mm:PinSocket_2x01_P2.54mm_Vertical, symbol Connector:Conn_01x02_Male
- added J13: 5V, Connector_PinSocket_2.54mm:PinSocket_2x01_P2.54mm_Vertical, symbol Connector:Conn_01x02_Male
- added R21: 1K, Resistor_SMD:R_0603_1608Metric_Pad0.98x0.95mm_HandSolder, symbol Device:R
- added R22, R23, R24: 10k, Resistor_SMD:R_0603_1608Metric_Pad0.98x0.95mm_HandSolder, symbol uven-mainboard-rescue:R-Device
- added TP13: TEMP_DRIVER_LED, custom_lib:TP420X150, symbol RCWCTE:RCWCTE
- added TP14: TEMP_CHAMBER0, custom_lib:TP420X150, symbol RCWCTE:RCWCTE
- added TP15: LED_SENS, custom_lib:TP420X150, symbol RCWCTE:RCWCTE
- added TP16: TEMP_DRIVER_TEC_CHAMBER, custom_lib:TP420X150, symbol RCWCTE:RCWCTE
- added TP17: TEMP_LED0, custom_lib:TP420X150, symbol RCWCTE:RCWCTE
- added TP18: TEMP_LED1, custom_lib:TP420X150, symbol RCWCTE:RCWCTE
- added TP19: SEL1, custom_lib:TP420X150, symbol RCWCTE:RCWCTE
- added TP20: SEL0, custom_lib:TP420X150, symbol RCWCTE:RCWCTE
- added TP21: LATCH, custom_lib:TP420X150, symbol RCWCTE:RCWCTE
- added TP22: CS, custom_lib:TP420X150, symbol RCWCTE:RCWCTE
- added TP23: MISO, custom_lib:TP420X150, symbol RCWCTE:RCWCTE
- added TP24: MOSI, custom_lib:TP420X150, symbol RCWCTE:RCWCTE
- added TP25: SCK, custom_lib:TP420X150, symbol RCWCTE:RCWCTE
- added TP26: LED_ENABLE, custom_lib:TP420X150, symbol RCWCTE:RCWCTE
- added TP27: LED_DIAG_ENABLE, custom_lib:TP420X150, symbol RCWCTE:RCWCTE
- added TP28: TEC0_DIAG_ENABLE, custom_lib:TP420X150, symbol RCWCTE:RCWCTE
- added TP29: TEC1_DIAG_ENABLE, custom_lib:TP420X150, symbol RCWCTE:RCWCTE
- added TP30: LED_LATCH, custom_lib:TP420X150, symbol RCWCTE:RCWCTE
- added TP31: TEC_LED_LATCH, custom_lib:TP420X150, symbol RCWCTE:RCWCTE
- added TP32: TEC_CHAMBER_LATCH, custom_lib:TP420X150, symbol RCWCTE:RCWCTE
- added TP33: TEMP_CHAMBER1, custom_lib:TP420X150, symbol RCWCTE:RCWCTE
- added TP34: TEMP_DRIVER_TEC_LED, custom_lib:TP420X150, symbol RCWCTE:RCWCTE
- renumbered 1 to 11111
Connections:
- net +3.3V: now also J12.1 (Pin_1)
- net +5V: now also D1.2 (A), J13.1 (Pin_1)
- net CS: now also TP22.1
- net GND: now also J12.2 (Pin_2), J13.2 (Pin_2), R21.2, R24.1
- net LATCH: now also TP21.1
- net LED0+: now also D2.2 (A)
- net LED0-: now also R22.2
- net LED1+: now also D3.2 (A)
- net LED1-: now also R23.2
- net LED_DIAG_ENABLE: now also TP27.1
- net LED_ENABLE: now also R24.2, TP26.1
- net LED_LATCH: now also TP30.1
- net LED_SENS: now also TP15.1
- net SEL0: now also TP20.1
- net SEL1: now also TP19.1
- net SPI_MISO: now also TP23.1
- net SPI_MOSI: now also TP24.1
- net SPI_SCK: now also TP25.1
- net TEC0_DIAG_ENABLE: now also TP28.1
- net TEC1_DIAG_ENABLE: now also TP29.1
- net TEC_CHAMBER_LATCH: now also TP32.1
- net TEC_LED_LATCH: now also TP31.1
- net TEMP_CHAMBER0: now also TP14.1
- net TEMP_CHAMBER1: now also TP33.1
- net TEMP_DRIVER_LED: now also TP13.1
- net TEMP_DRIVER_TEC_CHAMBER: now also TP16.1
- net TEMP_DRIVER_TEC_LED: now also TP34.1
- net TEMP_LED0: now also TP17.1
- net TEMP_LED1: now also TP18.1
- new net: D2.1 (K), R22.1
- new net: D1.1 (K), R21.1
- new net: D3.1 (K), R23.1
Other:
- moved on the sheet: C3, C4, C7, J3, J4, JP1, R5, R6, TH1, TP1, TP2, TP3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
