File: hardware/uven2-mk2-interface-board/uven2-mk2-interface-board.kicad_pcb (KiCad board)
At the start: 4 copper layers, 157 x 64 mm, 63 parts, among them J1 Chamber_Control, J10 LEDs_1, J2 TEMP_LEDS, J3 CHAMBER_FAN_0, J4 CHAMBER_FAN_1, J5 LED_FAN, J6 LED_ENABLE, J7 LED_ENABLE, J8 LEDs_0, J9 LEDs

Commit message: ordered on jlcpcb
Parts:
- added FID1: Fiducial, Fiducial:Fiducial_1mm_Dia_2.54mm_Outer_CopperTop, F.Cu at (110.5, 75.0)
- added FID2: Fiducial, Fiducial:Fiducial_1mm_Dia_2.54mm_Outer_CopperTop, F.Cu at (245.0, 75.0)
- added FID3: Fiducial, Fiducial:Fiducial_1mm_Dia_2.54mm_Outer_CopperTop, F.Cu at (245.0, 20.0)
