File: hardware/uven2-mk2-interface-board/uven2-mk2-interface-board.kicad_sch (KiCad schematic)
At the start: 63 parts, among them J1 Chamber_Control, J10 LEDs_1, J2 TEMP_LEDS, J3 CHAMBER_FAN_0, J4 CHAMBER_FAN_1, J5 LED_FAN, J6 LED_ENABLE, J7 LED_ENABLE, J8 LEDs_0, J9 LEDs

Commit message: ordered on jlcpcb
Parts:
- added FID1, FID2, FID3: Fiducial, Fiducial:Fiducial_1mm_Dia_2.54mm_Outer_CopperTop, symbol Mechanical:Fiducial
Changed lines of the file:
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@@
     (pin "1")
+  )
+  (symbol (lib_id "Mechanical:Fiducial") (at 126.365 178.435 0) (unit 1)
+    (in_bom yes) (on_board yes) (fields_autoplaced)
+    (property "Reference" "FID2" (id 0) (at 128.524 177.6003 0)
+      (effects (font (size 1.27 1.27)) (justify left))
+    )
+    (property "Value" "Fiducial" (id 1) (at 128.524 180.1372 0)
+      (effects (font (size 1.27 1.27)) (justify left))
+    )
+    (property "Footprint" "Fiducial:Fiducial_1mm_Dia_2.54mm_Outer_CopperTop" (id 2) (at 126.365 178.435 0)
+      (effects (font (size 1.27 1.27)) hide)
+    )
+    (property "Datasheet" "~" (id 3) (at 126.365 178.435 0)
+      (effects (font (size 1.27 1.27)) hide)
+    )
   )
   (symbol (lib_id "Power_Protection:SP0502BAHT") (at 54.61 170.18 0) (unit 1)
@@
     (pin "1")
   )
+  (symbol (lib_id "Mechanical:Fiducial") (at 126.365 186.055 0) (unit 1)
+    (in_bom yes) (on_board yes) (fields_autoplaced)
+    (property "Reference" "FID3" (id 0) (at 128.524 185.2203 0)
+      (effects (font (size 1.27 1.27)) (justify left))
+    )
+    (property "Value" "Fiducial" (id 1) (at 128.524 187.7572 0)
+      (effects (font (size 1.27 1.27)) (justify left))
+    )
+    (property "Footprint" "Fiducial:Fiducial_1mm_Dia_2.54mm_Outer_CopperTop" (id 2) (at 126.365 186.055 0)
+      (effects (font (size 1.27 1.27)) hide)
+    )
+    (property "Datasheet" "~" (id 3) (at 126.365 186.055 0)
+      (effects (font (size 1.27 1.27)) hide)
+    )
+  )
   (symbol (lib_id "power:GND") (at 158.75 68.58 270) (unit 1)
     (in_bom yes) (on_board yes)
@@
     (pin "1")
     (pin "2")
+  )
+  (symbol (lib_id "Mechanical:Fiducial") (at 126.365 170.815 0) (unit 1)
+    (in_bom yes) (on_board yes) (fields_autoplaced)
+    (property "Reference" "FID1" (id 0) (at 128.524 169.9803 0)
+      (effects (font (size 1.27 1.27)) (justify left))
+    )
+    (property "Value" "Fiducial" (id 1) (at 128.524 172.5172 0)
+      (effects (font (size 1.27 1.27)) (justify left))
+    )
+    (property "Footprint" "Fiducial:Fiducial_1mm_Dia_2.54mm_Outer_CopperTop" (id 2) (at 126.365 170.815 0)
+      (effects (font (size 1.27 1.27)) hide)
+    )
+    (property "Datasheet" "~" (id 3) (at 126.365 170.815 0)
+      (effects (font (size 1.27 1.27)) hide)
+    )
   )
   (symbol (lib_id "Mechanical:MountingHole") (at 125.73 109.22 0) (unit 1)
@@
       (reference "D32") (unit 1) (value "VESD16A2") (footprint "Package_TO_SOT_SMD:SOT-23")
     )
+    (path "/bf50b93b-d150-486b-953d-99999db03b48"
+      (reference "FID1") (unit 1) (value "Fiducial") (footprint "Fiducial:Fiducial_1mm_Dia_2.54mm_Outer_CopperTop")
+    )
+    (path "/6fa7c350-d764-4117-bc25-11d83a168714"
+      (reference "FID2") (unit 1) (value "Fiducial") (footprint "Fiducial:Fiducial_1mm_Dia_2.54mm_Outer_CopperTop")
+    )
+    (path "/a68f66d2-e655-4c7a-b2d1-f45d50de165d"
+      (reference "FID3") (unit 1) (value "Fiducial") (footprint "Fiducial:Fiducial_1mm_Dia_2.54mm_Outer_CopperTop")
+    )
     (path "/c129847e-9b37-44c9-982b-902ba2d73e39"
