File: hardware/uven2-mk3-cc-driver/uven2-mk3-cc-driver.kicad_sch (KiCad schematic)
At the start: 17 parts, among them J1 48VDC IN, J2 ADJ, J3 ENABLE, J4 LED, Q1 AO3401A, U2 LM3409HV

Commit message: cc driver test draft
Parts:
- removed D1: B1100-13-F, Diodes_SMD:D_SMA, symbol led-driver-rescue:D_Schottky_Small_ALT-led-driver-rescue
- removed J1: 48VDC IN, Pin_Headers:Pin_Header_Straight_1x02_Pitch2.54mm, symbol led-driver-rescue:CONN_01X02-led-driver-rescue
- removed J2: ADJ, Pin_Headers:Pin_Header_Straight_1x02_Pitch2.54mm, symbol led-driver-rescue:CONN_01X02-led-driver-rescue
- removed J3: ENABLE, Pin_Headers:Pin_Header_Straight_1x03_Pitch2.54mm, symbol led-driver-rescue:CONN_01X03-led-driver-rescue
- removed J4: LED, Pin_Headers:Pin_Header_Straight_1x02_Pitch2.54mm, symbol led-driver-rescue:CONN_01X02-led-driver-rescue
- added D2: SBT-10X-UV-A120-AH380-22, custom_lib:LED_SBT-10X-UV-A120-AH380-22, symbol SBT-10X-UV-A120-AH380-22:SBT-10X-UV-A120-AH380-22
- added D3: SS34, custom_lib:DIO_SS34, symbol SS34:SS34
- added H1, H2, H3, H4, H5, H6: MountingHole, MountingHole:MountingHole_2.2mm_M2, symbol Mechanical:MountingHole
- added J1: Conn_01x03_Pin, Connector_PinSocket_2.54mm:PinSocket_1x03_P2.54mm_Vertical, symbol Connector:Conn_01x03_Pin
- added J2: ADJ, Connector_PinSocket_2.54mm:PinSocket_1x02_P2.54mm_Vertical, symbol Connector:Conn_01x02_Socket
- added J3: current_measurement, Connector_PinHeader_2.54mm:PinHeader_1x02_P2.54mm_Vertical, symbol Connector:Conn_01x02_Pin
- C1: footprint Capacitors_SMD:CP_Elec_5x5.3 -> Capacitor_SMD:C_Elec_5x5.4
- C2, C3, C4: footprint Capacitors_SMD:C_0805 -> Capacitor_SMD:C_0603_1608Metric_Pad1.08x0.95mm_HandSolder
- C5: footprint Capacitors_SMD:C_1812 -> Capacitor_SMD:C_1812_4532Metric_Pad1.57x3.40mm_HandSolder
- L1: footprint Choke_SMD:Choke_SMD_7.3x7.3_H3.5 -> Inductor_SMD:L_7.3x7.3_H3.5
- R1: value 49.9kΩ -> 24kΩ; footprint Resistors_SMD:R_0805 -> Resistor_SMD:R_0805_2012Metric_Pad1.20x1.40mm_HandSolder
- R2: value 1.47kΩ -> 4.7kΩ; footprint Resistors_SMD:R_0805 -> Resistor_SMD:R_0805_2012Metric_Pad1.20x1.40mm_HandSolder
- R3, R4: footprint Resistors_SMD:R_0805 -> Resistor_SMD:R_0805_2012Metric_Pad1.20x1.40mm_HandSolder
- U2: footprint Housings_SSOP:MSOP-10-1EP_3x3mm_Pitch0.5mm -> custom_lib:IC_XTR111AIDGQR
Connections:
- net GND: now also D2.C, D2.EXP, D3.A, J1.2 (Pin_2), J2.1 (Pin_1)
- net VCC: now also J1.1 (Pin_1)
- net at L1.1, Q1.2 (S): now also D3.C
- net at C5.1, L1.2, R3.1: now also J3.2 (Pin_2)
- net at C2.2, U2.2 (IADJ): now also J2.2 (Pin_2)
- net ENABLE: now reaches U2.3 (EN)
- net ENABLE: now also J1.3 (Pin_3)
- new net: D2.A, J3.1 (Pin_1)
Other:
- moved on the sheet: C3

Commit message: ordered
Parts:
- removed C1: 3.3µF, Capacitor_SMD:C_Elec_5x5.4, symbol led-driver-rescue:C_Small-led-driver-rescue
- removed D3: SS34, custom_lib:DIO_SS34, symbol SS34:SS34
- added C1: 16SVP3R3M, custom_lib:CAP_16SVP3R3M, symbol 16SVP3R3M:16SVP3R3M
- added D1: SS54-HF, custom_lib:DIOM5025X220N, symbol SS54-HF:SS54-HF
- L1: footprint Inductor_SMD:L_7.3x7.3_H3.5 -> custom_lib:HPC-8040NV-100M
- R1, R2, R3: footprint Resistor_SMD:R_0805_2012Metric_Pad1.20x1.40mm_HandSolder -> Resistor_SMD:R_0603_1608Metric_Pad0.98x0.95mm_HandSolder
- R4: footprint Resistor_SMD:R_0805_2012Metric_Pad1.20x1.40mm_HandSolder -> Resistor_SMD:R_2512_6332Metric_Pad1.40x3.35mm_HandSolder
Connections:
- net GND: now also C1.2, D1.2
- net VCC: now also C1.1
- net at L1.1, Q1.2 (S): now also D1.1

Commit message: fix mosfet wrong orientation
Connections:
- net at R4.2, U2.7 (CSN): now also Q1.2 (S); no longer Q1.3 (D)
- net at D1.1, L1.1: now also Q1.3 (D); no longer Q1.2 (S)
Other:
- moved on the sheet: Q1
Changed lines of the file:
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@@
   (junction (at 179.07 73.66) (diameter 0) (color 0 0 0 0)
   )
+  (junction (at 190.5 88.9) (diameter 0) (color 0 0 0 0)
+  )
   (junction (at 190.5 100.33) (diameter 0) (color 0 0 0 0)
   )
@@
   (junction (at 141.605 104.14) (diameter 0) (color 0 0 0 0)
   )
-  (junction (at 190.5 88.9) (diameter 0) (color 0 0 0 0)
-  )
   (junction (at 134.62 78.74) (diameter 0) (color 0 0 0 0)
   )
@@
     (stroke (width 0) (type default))
   )
+  (wire (pts (xy 179.07 97.155) (xy 198.12 97.155))
+    (stroke (width 0) (type default))
+  )
   (wire (pts (xy 205.74 102.87) (xy 205.74 100.33))
     (stroke (width 0) (type default))
@@
     (stroke (width 0) (type default))
   )
+  (wire (pts (xy 179.07 93.98) (xy 179.07 97.155))
+    (stroke (width 0) (type default))
+  )
+  (wire (pts (xy 175.26 93.98) (xy 179.07 93.98))
+    (stroke (width 0) (type default))
+  )
   (wire (pts (xy 201.93 117.475) (xy 201.93 100.33))
     (stroke (width 0) (type default))
@@
     (stroke (width 0) (type default))
   )
-  (wire (pts (xy 182.88 93.98) (xy 175.26 93.98))
-    (stroke (width 0) (type default))
-  )
   (wire (pts (xy 175.26 88.9) (xy 190.5 88.9))
     (stroke (width 0) (type default))
@@
   )
   (wire (pts (xy 218.44 100.33) (xy 228.6 100.33))
+    (stroke (width 0) (type default))
+  )
+  (wire (pts (xy 198.12 97.155) (xy 198.12 93.98))
     (stroke (width 0) (type default))
   )
@@
     )
   )
-  (symbol (lib_id "Transistor_FET:AO3401A") (at 187.96 93.98 0) (unit 1)
+  (symbol (lib_id "Transistor_FET:AO3401A") (at 193.04 93.98 180) (unit 1)
     (in_bom yes) (on_board yes) (dnp no) (fields_autoplaced)
-    (property "Reference" "Q1" (at 193.167 92.7679 0)
-      (effects (font (size 1.27 1.27)) (justify left))
-    )
-    (property "Value" "AO3401A" (at 193.167 95.1921 0)
-      (effects (font (size 1.27 1.27)) (justify left))
-    )
-    (property "Footprint" "Package_TO_SOT_SMD:SOT-23" (at 193.04 95.885 0)
+    (property "Reference" "Q1" (at 187.8331 92.7679 0)
+      (effects (font (size 1.27 1.27)) (justify left))
+    )
+    (property "Value" "AO3401A" (at 187.8331 95.1921 0)
+      (effects (font (size 1.27 1.27)) (justify left))
+    )
+    (property "Footprint" "Package_TO_SOT_SMD:SOT-23" (at 187.96 92.075 0)
       (effects (font (size 1.27 1.27) italic) (justify left) hide)
     )
-    (property "Datasheet" "http://www.aosmd.com/pdfs/datasheet/AO3401A.pdf" (at 187.96 93.98 0)
+    (property "Datasheet" "http://www.aosmd.com/pdfs/datasheet/AO3401A.pdf" (at 193.04 93.98 0)
       (effects (font (size 1.27 1.27)) (justify left) hide)
     )
