File: hardware/uven2-mk3-led-array-100x/uven2-mk3-led-array-100x.kicad_sch (KiCad schematic)
At the start: 0 parts

Commit message: more layout
Parts:
- added J1, J2: TSM-150-01-S-DH, custom_lib:SAMTEC_TSM-150-01-S-DH, symbol TSM-150-01-S-DH:TSM-150-01-S-DH
Connections:
- new net ANODE_: J1.02, J1.04, J1.06, J1.08, J1.10, J1.12, J1.14, J1.16, J1.18, J1.20, J1.22, J1.24, J1.26, J1.28, J1.30, J1.32, J1.34, J1.36, J1.38, J1.40, J1.42, J1.44, J1.46, J1.48, J1.50, J1.52, J1.54, J1.56, J1.58, J1.60, J2.02, J2.04, J2.06, J2.08, J2.10, J2.100, J2.12, J2.14, J2.16, J2.18, J2.20, J2.22, J2.24, J2.26, J2.28, J2.30, J2.32, J2.34, J2.36, J2.38, J2.40, J2.42, J2.44, J2.46, J2.48, J2.50, J2.52, J2.54, J2.56, J2.58, J2.60, J2.62, J2.64, J2.66, J2.68, J2.70, J2.72, J2.74, J2.76, J2.78, J2.80, J2.82, J2.84, J2.86, J2.88, J2.90, J2.92, J2.94, J2.96, J2.98
- new net ANODE_14: J1.66
- new net ANODE_15: J1.76
- new net ANODE_29: J1.62
- new net ANODE_30: J1.70
- new net ANODE_31: J1.80
- new net ANODE_32: J1.86
- new net ANODE_33: J1.92
- new net ANODE_51: J1.68
- new net ANODE_52: J1.74
- new net ANODE_53: J1.82
- new net ANODE_54: J1.88
- new net ANODE_55: J1.94
- new net ANODE_56: J1.96
- new net ANODE_78: J1.64
- new net ANODE_79: J1.72
- new net ANODE_80: J1.78
- new net ANODE_81: J1.84
- new net ANODE_82: J1.90
- new net ANODE_83: J1.98
- new net ANODE_84: J1.100
- new net CATHODE_: J1.01, J1.03, J1.05, J1.07, J1.09, J1.11, J1.13, J1.15, J1.17, J1.19, J1.21, J1.23, J1.25, J1.27, J1.29, J1.31, J1.33, J1.35, J1.37, J1.39, J1.41, J1.43, J1.45, J1.47, J1.49, J1.51, J1.53, J1.55, J1.57, J1.59, J2.01, J2.03, J2.05, J2.07, J2.09, J2.11, J2.13, J2.15, J2.17, J2.19, J2.21, J2.23, J2.25, J2.27, J2.29, J2.31, J2.33, J2.35, J2.37, J2.39, J2.41, J2.43, J2.45, J2.47, J2.49, J2.51, J2.53, J2.55, J2.57, J2.59, J2.61, J2.63, J2.65, J2.67, J2.69, J2.71, J2.73, J2.75, J2.77, J2.79, J2.81, J2.83, J2.85, J2.87, J2.89, J2.91, J2.93, J2.95, J2.97, J2.99
- new net CATHODE_14: J1.65
- new net CATHODE_15: J1.75
- new net CATHODE_29: J1.61
- new net CATHODE_30: J1.69
- new net CATHODE_31: J1.79
- new net CATHODE_32: J1.85
- new net CATHODE_33: J1.91
- new net CATHODE_51: J1.67
- new net CATHODE_52: J1.73
- new net CATHODE_53: J1.81
- new net CATHODE_54: J1.87
- new net CATHODE_55: J1.93
- new net CATHODE_56: J1.95
- new net CATHODE_78: J1.63
- new net CATHODE_79: J1.71
- new net CATHODE_80: J1.77
- new net CATHODE_81: J1.83
- new net CATHODE_82: J1.89
- new net CATHODE_83: J1.97
- new net CATHODE_84: J1.99

Commit message: more layout
Connections:
- net ANODE_0: now also J1.48
- net ANODE_1: now also J2.76
- net ANODE_10: now also J1.24
- net ANODE_11: now also J1.32
- net ANODE_12: now also J1.44
- net ANODE_13: now also J1.56
- net ANODE_16: now also J2.34
- net ANODE_17: now also J2.20
- net ANODE_18: now also J2.24
- net ANODE_19: now also J2.44
- net ANODE_2: now also J1.40
- net ANODE_20: now also J2.54
- net ANODE_21: now also J2.68
- net ANODE_22: now also J2.78
- net ANODE_23: now also J2.100
- net ANODE_24: now also J1.16
- net ANODE_25: now also J1.22
- net ANODE_26: now also J1.30
- net ANODE_27: now also J1.38
- net ANODE_28: now also J1.52
- net ANODE_3: now also J1.50
- net ANODE_34: now also J2.08
- net ANODE_35: now also J2.14
- net ANODE_36: now also J2.30
- net ANODE_37: now also J2.40
- net ANODE_38: now also J2.50
- net ANODE_39: now also J2.62
- net ANODE_4: now also J1.60
- net ANODE_40: now also J2.70
- net ANODE_41: now also J2.80
- net ANODE_42: now also J2.92
- net ANODE_43: now also J1.06
- net ANODE_44: now also J1.10
- net ANODE_45: now also J1.14
- net ANODE_46: now also J1.20
- net ANODE_47: now also J1.28
- net ANODE_48: now also J1.36
- net ANODE_49: now also J1.46
- net ANODE_5: now also J2.36
- net ANODE_50: now also J1.58
- net ANODE_57: now also J2.04
- net ANODE_58: now also J2.10
- net ANODE_59: now also J2.16
- net ANODE_6: now also J2.22
- net ANODE_60: now also J2.28
- net ANODE_61: now also J2.38
- net ANODE_62: now also J2.48
- net ANODE_63: now also J2.56
- net ANODE_64: now also J2.64
- net ANODE_65: now also J2.72
- net ANODE_66: now also J2.84
- net ANODE_67: now also J2.90
- net ANODE_68: now also J2.96
- net ANODE_69: now also J1.02
- net ANODE_7: now also J2.46
- net ANODE_70: now also J1.04
- net ANODE_71: now also J1.08
- net ANODE_72: now also J1.12
- net ANODE_73: now also J1.18
- net ANODE_74: now also J1.26
- net ANODE_75: now also J1.34
- net ANODE_76: now also J1.42
- net ANODE_77: now also J1.54
- net ANODE_8: now also J2.60
- net ANODE_85: now also J2.02
- net ANODE_86: now also J2.06
- net ANODE_87: now also J2.12
- net ANODE_88: now also J2.18
- net ANODE_89: now also J2.26
- net ANODE_9: now also J2.86
- net ANODE_90: now also J2.32
- net ANODE_91: now also J2.42
- net ANODE_92: now also J2.52
- net ANODE_93: now also J2.58
- net ANODE_94: now also J2.66
- net ANODE_95: now also J2.74
- net ANODE_96: now also J2.82
- net ANODE_97: now also J2.88
- net ANODE_98: now also J2.94
- net ANODE_99: now also J2.98
- net CATHODE_0: now also J1.47
- net CATHODE_1: now also J2.75
- net CATHODE_10: now also J1.23
- net CATHODE_11: now also J1.31
- net CATHODE_12: now also J1.43
- net CATHODE_13: now also J1.55
- net CATHODE_16: now also J2.33
- net CATHODE_17: now also J2.19
- net CATHODE_18: now also J2.23
- net CATHODE_19: now also J2.43
- net CATHODE_2: now also J1.39
- net CATHODE_20: now also J2.53
- net CATHODE_21: now also J2.67
- net CATHODE_22: now also J2.77
- net CATHODE_23: now also J2.99
- net CATHODE_24: now also J1.15
- net CATHODE_25: now also J1.21
- net CATHODE_26: now also J1.29
- net CATHODE_27: now also J1.37
- net CATHODE_28: now also J1.51
- net CATHODE_3: now also J1.49
- net CATHODE_34: now also J2.07
- net CATHODE_35: now also J2.13
- net CATHODE_36: now also J2.29
- net CATHODE_37: now also J2.39
- net CATHODE_38: now also J2.49
- net CATHODE_39: now also J2.61
- net CATHODE_4: now also J1.59
- net CATHODE_40: now also J2.69
- net CATHODE_41: now also J2.79
- net CATHODE_42: now also J2.91
- net CATHODE_43: now also J1.05
- net CATHODE_44: now also J1.09
- net CATHODE_45: now also J1.13
- net CATHODE_46: now also J1.19
- net CATHODE_47: now also J1.27
- net CATHODE_48: now also J1.35
- net CATHODE_49: now also J1.45
- net CATHODE_5: now also J2.35
- net CATHODE_50: now also J1.57
- net CATHODE_57: now also J2.03
- net CATHODE_58: now also J2.09
- net CATHODE_59: now also J2.15
- net CATHODE_6: now also J2.21
- net CATHODE_60: now also J2.27
- net CATHODE_61: now also J2.37
- net CATHODE_62: now also J2.47
- net CATHODE_63: now also J2.55
- net CATHODE_64: now also J2.63
- net CATHODE_65: now also J2.71
- net CATHODE_66: now also J2.83
- net CATHODE_67: now also J2.89
- net CATHODE_68: now also J2.95
- net CATHODE_69: now also J1.01
- net CATHODE_7: now also J2.45
- net CATHODE_70: now also J1.03
- net CATHODE_71: now also J1.07
- net CATHODE_72: now also J1.11
- net CATHODE_73: now also J1.17
- net CATHODE_74: now also J1.25
- net CATHODE_75: now also J1.33
- net CATHODE_76: now also J1.41
- net CATHODE_77: now also J1.53
- net CATHODE_8: now also J2.59
- net CATHODE_85: now also J2.01
- net CATHODE_86: now also J2.05
- net CATHODE_87: now also J2.11
- net CATHODE_88: now also J2.17
- net CATHODE_89: now also J2.25
- net CATHODE_9: now also J2.85
- net CATHODE_90: now also J2.31
- net CATHODE_91: now also J2.41
- net CATHODE_92: now also J2.51
- net CATHODE_93: now also J2.57
- net CATHODE_94: now also J2.65
- net CATHODE_95: now also J2.73
- net CATHODE_96: now also J2.81
- net CATHODE_97: now also J2.87
- net CATHODE_98: now also J2.93
- net CATHODE_99: now also J2.97
- removed net ANODE_: J1.02, J1.04, J1.06, J1.08, J1.10, J1.12, J1.14, J1.16, J1.18, J1.20, J1.22, J1.24, J1.26, J1.28, J1.30, J1.32, J1.34, J1.36, J1.38, J1.40, J1.42, J1.44, J1.46, J1.48, J1.50, J1.52, J1.54, J1.56, J1.58, J1.60, J2.02, J2.04, J2.06, J2.08, J2.10, J2.100, J2.12, J2.14, J2.16, J2.18, J2.20, J2.22, J2.24, J2.26, J2.28, J2.30, J2.32, J2.34, J2.36, J2.38, J2.40, J2.42, J2.44, J2.46, J2.48, J2.50, J2.52, J2.54, J2.56, J2.58, J2.60, J2.62, J2.64, J2.66, J2.68, J2.70, J2.72, J2.74, J2.76, J2.78, J2.80, J2.82, J2.84, J2.86, J2.88, J2.90, J2.92, J2.94, J2.96, J2.98
- removed net CATHODE_: J1.01, J1.03, J1.05, J1.07, J1.09, J1.11, J1.13, J1.15, J1.17, J1.19, J1.21, J1.23, J1.25, J1.27, J1.29, J1.31, J1.33, J1.35, J1.37, J1.39, J1.41, J1.43, J1.45, J1.47, J1.49, J1.51, J1.53, J1.55, J1.57, J1.59, J2.01, J2.03, J2.05, J2.07, J2.09, J2.11, J2.13, J2.15, J2.17, J2.19, J2.21, J2.23, J2.25, J2.27, J2.29, J2.31, J2.33, J2.35, J2.37, J2.39, J2.41, J2.43, J2.45, J2.47, J2.49, J2.51, J2.53, J2.55, J2.57, J2.59, J2.61, J2.63, J2.65, J2.67, J2.69, J2.71, J2.73, J2.75, J2.77, J2.79, J2.81, J2.83, J2.85, J2.87, J2.89, J2.91, J2.93, J2.95, J2.97, J2.99

Commit message: layout almost finished
Parts:
- added H1, H10, H11, H12, H13, H14, H15, H16, H2, H3, H4, H5, H6, H7, H8, H9: MountingHole_Pad, MountingHole:MountingHole_3.2mm_M3_DIN965_Pad, symbol Mechanical:MountingHole_Pad
- added J3: TSM-104-01-L-DH, custom_lib:SAMTEC_TSM-104-01-L-DH, symbol TSM-104-01-L-DH:TSM-104-01-L-DH
- added TH1, TH2, TH3, TH4: Thermistor_NTC, Resistor_SMD:R_0805_2012Metric, symbol Device:Thermistor_NTC
Connections:
- new net: J3.07, TH2.1
- new net: J3.05, TH2.2
- new net: J3.04, TH3.1
- new net: J3.02, TH3.2
- new net: J3.01, TH1.2
- new net: J3.03, TH1.1
- new net: J3.06, TH4.2
- new net: J3.08, TH4.1
- new net GNDA: H1.1, H10.1, H11.1, H12.1, H13.1, H14.1, H15.1, H16.1, H2.1, H3.1, H4.1, H5.1, H6.1, H7.1, H8.1, H9.1
